File: philips_led_bulb.kicad_sch (KiCad schematic)
At the start: 21 parts, among them J1 Mains (E27 base), U1 KP18106WPA

Commit message: Add C1 value: 5.6uF 400V (Yunxing CD11-H)
Co-Authored-By: Claude Opus 5.5 <noreply@anthropic.com>
Claude-Session: https://claude.ai/code/session_01DkF4XRCCz81Qun3gAk33U7
Parts:
- C1: value Elcap (in base, value ?) -> 5.6uF 400V
Other:
- note added: "F1 and C1 are off-board (in the E27 base). C1: Yunxing CD11-H 5.6uF 400V 105C."
- note removed: "F1 and C1 are off-board (in the E27 base). C1 value not read yet."
Changed lines of the file:
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@@
 		)
 	)
-	(text "F1 and C1 are off-board (in the E27 base). C1 value not read yet."
+	(text "F1 and C1 are off-board (in the E27 base). C1: Yunxing CD11-H 5.6uF 400V 105C."
 		(exclude_from_sim no)
 		(at 25.4 178.435 0)
@@
 			)
 		)
-		(property "Value" "Elcap (in base, value ?)"
+		(property "Value" "5.6uF 400V"
 			(at 121.92 87.63 0)
 			(show_name no)
